Commit message: Add files via upload

File: urdf/common.urdf.xacro (robot description, xacro)
@@ -7,6 +7,6 @@
   <xacro:macro name="box_inertia" params="m x y z">
     <inertia ixx="${m*(y*y+z*z)/12}" ixy = "0" ixz = "0"
-             iyy="${m*(x*x+z*z)/12}" iyz = "0"
-             izz="${m*(x*x+z*z)/12}" />
+             iyy="${m*(z*z+x*x)/12}" iyz = "0"
+             izz="${m*(x*x+y*y)/12}" />
   </xacro:macro>
   <xacro:macro name="cylinder_inertia" params="m r h">

File: urdf/model01.urdf.xacro (robot description, xacro)
@@ -14,4 +14,5 @@
         <box size="0.069 0.138 0.050"/>
       </geometry>
+      <material name="White" />
     </visual>
     <inertial>
@@ -37,4 +38,5 @@
         <cylinder radius="0.069" length="0.172" />
       </geometry>
+      <material name="White" />
     </visual>
     <inertial>
